Commit message: temp2

File: resources/robots/lmf2/model.urdf (robot description, URDF)
Before this commit: robot quadrotor, 5 links, 4 joints
Joints:
- joint base_link_to_back_left_prop: origin xyz=-0.100 0.100 0 -> xyz=-0.0900 0.0900 0
- joint base_link_to_back_right_prop: origin xyz=-0.100 -0.100 0 -> xyz=-0.0900 -0.0900 0
- joint base_link_to_front_left_prop: origin xyz=0.100 0.100 0 -> xyz=0.0900 0.0900 0
- joint base_link_to_front_right_prop: origin xyz=0.100 -0.100 0 -> xyz=0.0900 -0.0900 0
